File: Module/Abstimmspannungs-Modul/Abstimmspannungs-Modul.kicad_pcb (KiCad board)
At the start: 2 copper layers, 60 x 60 mm, 20 parts, among them IC501 TCA530, J1 Conn_01x09, P512 1k, P516 100k

Commit message: A bunch of new modules added.
Parts:
- C502, C503: value 1µF -> 1µ; footprint Capacitors_THT:C_Rect_L4.6mm_W5.5mm_P2.50mm_MKS02_FKP02 -> Capacitor_THT:C_Rect_L4.6mm_W5.5mm_P2.50mm_MKS02_FKP02
- C504: value 22µF -> 22µ; footprint Capacitors_THT:CP_Radial_D5.0mm_P2.00mm -> Capacitor_THT:CP_Radial_D5.0mm_P2.00mm
- C506, C507: value 1nF -> 1n; footprint Capacitors_THT:C_Disc_D5.0mm_W2.5mm_P5.00mm -> Capacitor_THT:C_Disc_D4.3mm_W1.9mm_P5.00mm
- IC501: footprint Housings_DIP:DIP-16_W7.62mm_LongPads -> Package_DIP:DIP-16_W7.62mm
- J1: footprint Abstimmspannungs-Modul:Connector_01x09_5mm -> Library:Connector_01x09_5mm
- P512, P516: footprint Potentiometers:Potentiometer_Trimmer_Piher_PT-15h5_Vertical_Px5.0mm_Py10.0mm -> Potentiometer_THT:Potentiometer_Piher_PT-15-H05_Horizontal
- R501, R502, R504, R506, R508, R511, R512, R513, R514, R516, R517: footprint Resistors_THT:R_Axial_DIN0207_L6.3mm_D2.5mm_P10.16mm_Horizontal -> Resistor_THT:R_Axial_DIN0207_L6.3mm_D2.5mm_P10.16mm_Horizontal
- moved R504 31.7 mm to (88.8, 64.8)
- moved C504 27.0 mm to (83.8, 50.5)
- moved R514 25.2 mm to (39.8, 80.0), turned to 90 degrees
- moved R508 15.5 mm to (39.8, 64.8)
- moved C502 14.1 mm to (73.6, 65.5), turned to -90 degrees
- moved R513 11.3 mm to (44.8, 80.0)
- moved C506 8.29 mm to (71.8, 55.6)
- moved IC501 7.53 mm to (60.5, 55.6)
- moved C507 6.80 mm to (56.8, 55.6)
- moved C503 5.32 mm to (73.6, 73.5), turned to 90 degrees
- moved R511 3.76 mm to (49.8, 80.0)
- moved R517 3.76 mm to (54.8, 80.0)
- moved R506 3.75 mm to (83.8, 54.7)
- moved R501 1.27 mm to (88.8, 80.0)
- moved R502 1.27 mm to (83.8, 80.0)
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Routing:
- net GND: track 187.7 -> 0.00 mm, vias 1 -> 0
- net TIMING: track 120.4 -> 31.3 mm
- net MUTING: track 119.2 -> 33.2 mm, vias 0 -> 1
- net +15V: track 108.2 -> 46.3 mm, vias 0 -> 1
- net Net-(P512-Pad3): track 43.4 -> 11.7 mm
- net OUT_BOTTOM: track 63.6 -> 75.3 mm, vias 0 -> 1
- net +45V: track 17.5 -> 27.5 mm
- net TCA530_P8: track 46.7 -> 37.7 mm
- net TCA530_P11: track 28.4 -> 23.6 mm
- net OUT_TOP: track 22.5 -> 18.9 mm
- net TCA530_P14: track 14.1 -> 17.5 mm
- net TCA530_P6: track 58.2 -> 55.1 mm
- net TCA530_P10: track 18.7 -> 17.6 mm
- net AFC_02: track 7.47 -> 8.24 mm
- net AFC_01: track 7.47 -> 8.24 mm
- added copper zone on B.Cu, net GND
Other:
- net class Default removed
- board text added: "+15V"
- board text added: "+45V"
- board text added: "A.O."
- board text added: "A.U."
- board text added: "AFC"
- board text added: "GND"
- board text added: "MUTE"
- board text added: "TIMINIG"
