File: Module/Anzeige-Modul - 7140+9240+9241/hardware/Anzeige-Modul.kicad_pcb (KiCad board)
At the start: 2 copper layers, 137 x 102 mm, 55 parts, among them J1 Conn_01x09_Male, J3 Conn_02x03_Counter_Clockwise, J5 Conn_01x13_Male, J6 Conn_01x16_Male, Q11 BC847, Q21 BC847, Q31 BC847, Q41 BC847, Q51 BC847, Q61 BC847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

Commit message: A bunch of new modules added.
Parts:
- removed REF** (x2): MountingHole_3.5mm, Mounting_Holes:MountingHole_3.5mm
- C1, C2, C3, C4, C5, C6, C7: footprint Capacitors_SMD:C_0805 -> Capacitor_SMD:C_0805_2012Metric
- J1: footprint saba_9240_frontend:Pad_Array_3.81mm -> Anzeige-Modul:PadArray_3.81mm_01x09
- J3: footprint Pin_Headers:Pin_Header_Straight_2x03_Pitch2.54mm -> Connector_PinHeader_2.54mm:PinHeader_2x03_P2.54mm_Vertical
- J5: footprint saba_9240_frontend:Pad_Array_2.54mm_1x13 -> Anzeige-Modul:PadArray_2.54mm_01x13
- Q11, Q21, Q31, Q41, Q51, Q61, Q71: footprint TO_SOT_Packages_SMD:SOT-23 -> Package_TO_SOT_SMD:SOT-23
- R1, R11, R12, R13, R21, R22, R23, R31, R32, R33, R41, R42, R43, R51, R52, R53, R61, R63, R71, R72: footprint Resistors_SMD:R_0805 -> Resistor_SMD:R_0805_2012Metric
- SW1, SW2, SW3, SW4, SW5, SW6: footprint saba_9240_frontend:saba_92xx_push_button -> Anzeige-Modul:SW_PUSH_DPDT
- U1: footprint TO_SOT_Packages_SMD:SOT-89-3 -> Package_TO_SOT_SMD:SOT-89-3
- U2: footprint Housings_QFP:TQFP-32_7x7mm_Pitch0.8mm -> Package_QFP:TQFP-32_7x7mm_P0.8mm
- moved R1 6.78 mm to (107.0, 94.2)
- moved C4 2.50 mm to (111.3, 78.0)
- moved C6 1.38 mm to (107.0, 92.0), turned to 0 degrees
- moved C7 1.14 mm to (110.5, 92.0), turned to 0 degrees
- moved C1 0.25 mm to (98.5, 69.2)
- moved C2 0.25 mm to (101.5, 69.2)
- moved U1 0.17 mm to (100.0, 74.2)
Connections:
- J6 pad 10: Net-(J6-Pad10) -> unconnected-(J6-Pad10)
- J6 pad 11: Net-(J6-Pad11) -> unconnected-(J6-Pad11)
- J6 pad 8: Net-(J6-Pad8) -> unconnected-(J6-Pad8)
- U2 pad 1: Net-(U2-Pad1) -> unconnected-(U2-Pad1)
- U2 pad 19: Net-(U2-Pad19) -> unconnected-(U2-Pad19)
- U2 pad 2: Net-(U2-Pad2) -> unconnected-(U2-Pad2)
- U2 pad 22: Net-(U2-Pad22) -> unconnected-(U2-Pad22)
- U2 pad 23: Net-(U2-Pad23) -> unconnected-(U2-Pad23)
- U2 pad 25: Net-(U2-Pad25) -> unconnected-(U2-Pad25)
- U2 pad 7: Net-(U2-Pad7) -> unconnected-(U2-Pad7)
- U2 pad 8: Net-(U2-Pad8) -> unconnected-(U2-Pad8)
Routing:
- net IMPULS: track 88.5 -> 74.8 mm
- net +5V: track 65.5 -> 52.1 mm, vias 0 -> 1
- net GND: track 39.7 -> 28.0 mm
- net +12V: track 150.9 -> 145.2 mm, vias 1 -> 3
- net RESET: track 23.7 -> 29.4 mm, vias 1 -> 2
- net CLK: track 15.2 -> 14.4 mm
Other:
- outline, holes or cut-outs redrawn
- net class Default removed
- board text added: "Rev. B 2023-11-25 Yannick Bock"
- board text removed: "Rev. A 2022-03-30 Yannick Bock"
