File: Module/Impuls-Modul/Impuls-Modul.kicad_pcb (KiCad board)
At the start: 2 copper layers, 68.5 x 70 mm, 26 parts, among them J1 Conn_01x13, T772 BC558B, T774 BC548C, T777 BC558B, T781 BC548C, T788 BC558B, T792 BC327

Commit message: A bunch of new modules added.
Parts:
- C772: footprint Capacitors_THT:CP_Radial_D6.3mm_P2.50mm -> Capacitor_THT:CP_Radial_D6.3mm_P2.50mm
- C784, C797: footprint Capacitors_THT:C_Rect_L7.0mm_W2.0mm_P5.00mm -> Capacitor_THT:C_Rect_L7.0mm_W2.0mm_P5.00mm
- R771, R772, R773, R774, R776, R777, R778, R781, R786, R787, R788, R791, R793, R794: footprint Resistors_THT:R_Axial_DIN0207_L6.3mm_D2.5mm_P10.16mm_Horizontal -> Resistor_THT:R_Axial_DIN0207_L6.3mm_D2.5mm_P10.16mm_Horizontal
- R782: value 47k -> 4.7k; footprint Resistors_THT:R_Axial_DIN0207_L6.3mm_D2.5mm_P10.16mm_Horizontal -> Resistor_THT:R_Axial_DIN0207_L6.3mm_D2.5mm_P10.16mm_Horizontal
- T772, T777, T788: value BC558B -> BC557; footprint TO_SOT_Packages_THT:TO-92_Molded_Wide_Oval -> Package_TO_SOT_THT:TO-92_Wide
- T774, T781: value BC548C -> BC547; footprint TO_SOT_Packages_THT:TO-92_Molded_Wide_Oval -> Package_TO_SOT_THT:TO-92_Wide
- T792: footprint TO_SOT_Packages_THT:TO-92_Molded_Wide_Oval -> Package_TO_SOT_THT:TO-92_Wide
- moved C772 38.7 mm to (58.8, 72.5), turned to 0 degrees
- moved C784 5.83 mm to (62.5, 80.0)
- moved D794 5.24 mm to (78.8, 69.8)
- moved R771 5.24 mm to (41.2, 69.8)
- moved R772 5.24 mm to (36.2, 80.0)
- moved R776 5.24 mm to (46.2, 69.8)
- moved R777 5.24 mm to (51.2, 80.0)
- moved R782 5.24 mm to (68.8, 69.8)
- moved R788 5.24 mm to (73.8, 69.8)
- moved R791 5.24 mm to (83.8, 69.8)
- moved R793 5.24 mm to (73.8, 56.8)
- moved T774 5.24 mm to (41.3, 38.6)
- moved T781 5.24 mm to (51.3, 38.6)
- moved R773 5.24 mm to (41.2, 46.7)
- moved R774 5.24 mm to (36.2, 46.7)
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Routing:
- net GND: track 243.7 -> 0.00 mm
- net P2: track 76.2 -> 65.0 mm
- net +12V: track 153.5 -> 143.1 mm, vias 0 -> 1
- net P7: track 63.8 -> 54.3 mm
- net P4: track 31.6 -> 26.0 mm
- net P6: track 57.9 -> 52.3 mm
- net P11: track 13.3 -> 9.28 mm
- net P10: track 13.3 -> 9.28 mm
- net P5: track 13.9 -> 11.1 mm
- net P1: track 48.9 -> 46.7 mm
- net Net-(C784-Pad1): track 5.00 -> 6.25 mm
- net Net-(T792-B): track 6.54 -> 5.50 mm
- added copper zone on B.Cu, net GND
Other:
- net class Default removed
- board text added: "+12V"
- board text added: "GND"
