File: Module/Relais-Modul/Relais-Modul.kicad_pcb (KiCad board)
At the start: 2 copper layers, 68.5 x 70 mm, 30 parts, among them J1 Conn_01x13, T674 BC548C, T681 BC558B, T684 BC558B, T691 BC635

Commit message: A bunch of new modules added.
Parts:
- C681: value 2.2µF -> 2.2µ; footprint Capacitors_THT:CP_Radial_D5.0mm_P2.50mm -> Capacitor_THT:CP_Radial_D5.0mm_P2.50mm
- C686: value 100µF -> 100µ; footprint Capacitors_THT:CP_Radial_D6.3mm_P2.50mm -> Capacitor_THT:CP_Radial_D6.3mm_P2.50mm
- D1: value 1N4001 -> 1N4148; footprint Diode_THT:D_DO-41_SOD81_P7.62mm_Horizontal -> Diode_THT:D_DO-35_SOD27_P7.62mm_Horizontal
- D671, D672, D676, D677: footprint Diode_THT:D_DO-41_SOD81_P12.70mm_Horizontal -> Diode_THT:D_DO-41_SOD81_P10.16mm_Horizontal
- L1, L2: footprint Inductors_THT:L_Radial_D8.7mm_P5.00mm_Fastron_07HCP -> Inductor_THT:L_Radial_D8.7mm_P5.00mm_Fastron_07HCP
- R1, R2: footprint Resistors_THT:R_Axial_DIN0516_L15.5mm_D5.0mm_P7.62mm_Vertical -> Resistor_THT:R_Axial_DIN0516_L15.5mm_D5.0mm_P7.62mm_Vertical
- R671, R673, R674, R676, R678, R681, R682, R683, R684, R686, R687, R691: footprint Resistors_THT:R_Axial_DIN0207_L6.3mm_D2.5mm_P10.16mm_Horizontal -> Resistor_THT:R_Axial_DIN0207_L6.3mm_D2.5mm_P10.16mm_Horizontal
- R688: value 15 -> 47; footprint Resistors_THT:R_Axial_DIN0207_L6.3mm_D2.5mm_P10.16mm_Horizontal -> Resistor_THT:R_Axial_DIN0207_L6.3mm_D2.5mm_P10.16mm_Horizontal
- T674: value BC548C -> BC547; footprint TO_SOT_Packages_THT:TO-92_Molded_Wide_Oval -> Package_TO_SOT_THT:TO-92_Wide
- T681, T684: value BC558B -> BC557; footprint TO_SOT_Packages_THT:TO-92_Molded_Wide_Oval -> Package_TO_SOT_THT:TO-92_Wide
- T691: value BC635 -> BC639; footprint TO_SOT_Packages_THT:TO-92_Molded_Wide_Oval -> Package_TO_SOT_THT:TO-92_Wide
- moved R688 44.4 mm to (35.8, 39.5), turned to -90 degrees
- moved R687 27.6 mm to (55.8, 49.7), turned to 90 degrees
- moved C681 25.3 mm to (60.8, 35.8), turned to 90 degrees
- moved C686 22.5 mm to (88.2, 45.5)
- moved T691 17.0 mm to (75.8, 33.7), turned to 180 degrees
- moved R686 15.3 mm to (55.8, 54.7), turned to -90 degrees
- moved R691 15.1 mm to (30.8, 64.8)
- moved R682 13.0 mm to (60.8, 49.7)
- moved R671 12.5 mm to (45.8, 80.0)
- moved R674 11.2 mm to (45.8, 54.7), turned to -90 degrees
- moved R673 9.15 mm to (45.8, 49.7)
- moved R678 7.29 mm to (40.8, 39.5), turned to -90 degrees
- moved R683 5.62 mm to (50.8, 54.7), turned to -90 degrees
- moved T674 3.51 mm to (38.2, 57.3)
- moved T681 2.63 mm to (45.7, 35.3), turned to 0 degrees
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Connections:
- net P1 renamed OUT-R
- net P10 renamed +12V
- net P2 renamed IN-R
- net P3 renamed OUT-L
- net P5 renamed IN-L
- net P9 renamed GND
- RL691 pad 12: Net-(RL691-Pad12) -> unconnected-(RL691-Pad12)
- RL691 pad 22: Net-(RL691-Pad22) -> unconnected-(RL691-Pad22)
Routing:
- net GND: track 141.9 -> 0.00 mm, vias 1 -> 0
- net +12V: track 109.7 -> 80.9 mm, vias 0 -> 1
- net Net-(D1-K): track 91.5 -> 70.8 mm, vias 2 -> 0
- net Net-(T691-B): track 28.4 -> 8.83 mm
- net P11: track 41.4 -> 25.2 mm
- net Net-(D1-A): track 24.1 -> 9.80 mm
- net Net-(D671-K): track 22.1 -> 10.0 mm
- net Net-(T681-B): track 16.0 -> 25.2 mm
- net Net-(T684-B): track 38.6 -> 45.7 mm
- net P8: track 34.7 -> 29.1 mm
- net Net-(T674-C): track 14.2 -> 8.67 mm
- net Net-(T681-C): track 14.3 -> 9.25 mm
- net P7: track 25.3 -> 20.3 mm
- net Net-(T674-B): track 20.1 -> 24.3 mm
- net Net-(T684-C): track 4.43 -> 7.57 mm
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- added copper zone on B.Cu, net GND
Other:
- net class Default removed
- board text added: "+12V"
- board text added: "GND"
- board text added: "JLCJLCJLCJLC"
- board text added: "L"
- board text added: "R"
