File: Module/Tipp-Tasten-Modul/hardware/Tipp-Tasten-Modul.kicad_pcb (KiCad board)
At the start: 2 copper layers, 205 x 49.5 mm, 39 parts, among them J1 Conn_01x09_Female, J10 Conn_01x01_Female, J2 Conn_01x05_Female, J3 Conn_01x05_Female, J4 Conn_01x01_Female, J5 Conn_01x01_Female, J6 Conn_01x01_Female, J8 Conn_01x01_Female, J9 Conn_01x01_Female, M2 MountingHole_3.5mm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

Commit message: A bunch of new modules added.
Other:
- net class Default removed
- board text removed: "Rev. A 2022-03-30 Yannick Bock"
