File: Module/Tipp-Tasten-Modul/hardware/Tipp-Tasten-Modul.kicad_sch (KiCad schematic)
At the start: 37 parts, among them J1 Conn_01x09_Female, J10 Conn_01x01_Female, J2 Conn_01x05_Female, J3 Conn_01x05_Female, J4 Conn_01x01_Female, J5 Conn_01x01_Female, J6 Conn_01x01_Female, J8 Conn_01x01_Female, J9 Conn_01x01_Female, SW1032 SW_Push_Dual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

Commit message: AZ553: LEDS added to BOM / Anzeige-Modul: Added additional Monting-Holes / Tipp-Tasten-Modul: Modified Push-Button Footprint
Parts:
- removed J9: Conn_01x01_Female, Wire_Pads:SolderWirePad_single_1-5mmDrill, symbol Connector:Conn_01x01_Female
- D1181, D1182, D1183, D1184, D1186, D1187, D1188, D1191, D1192: footprint LEDs:LED_D3.0mm -> LED_THT:LED_D3.0mm
- J1: footprint Tipp-Tasten-Modul:SolderWirePad_09_2.54mm -> Library:Conn_01x09; symbol Connector:Conn_01x09_Female -> Connector_Generic:Conn_01x09
- J10, J4, J5, J6, J8: symbol Connector:Conn_01x01_Female -> Connector_Generic:Conn_01x01
- J2, J3: footprint Tipp-Tasten-Modul:SolderWirePad_05_2.54mm -> Library:Conn_01x05; symbol Connector:Conn_01x05_Female -> Connector_Generic:Conn_01x05
- SW1032: footprint saba_924x_tipp-tasten-modul:saba_92xx_push_button -> Library:SW__PUSH_DPDT
- SW1181, SW1182, SW1183, SW1184, SW1186, SW1187, SW1188, SW1191: footprint Tipp-Tasten-Modul:SW_PUSH_DPDT -> Library:SW__PUSH_DPDT
